Commit message: Enhance camera calibration handling and update tmuxp configurations for improved node execution

File: earthrovers_description/src/description/frodobot.urdf (robot description, URDF)
Before this commit: robot rover, 6 links, 5 joints
Joints:
- joint front_camera_joint: origin xyz=0.013 0.0 0.561 rpy=0 0 0 -> xyz=0.013 0.0 0.561 rpy=-1.57079632679 0.0 -1.57079632679
